File: X88J.kicad_pcb (KiCad board)
At the start: 2 copper layers, 344 x 117.5 mm, 238 parts, among them J1 SM04B-SRSS-TB, J2 TC2030_SWD, U1 XC6206P332MR, U2 STM32F072CBT6

Commit message: Rotate JST to face alphas
Parts:
- turned J1 to 90 degrees
Routing:
- net D+: track 68.9 -> 77.5 mm
- net D-: track 68.9 -> 77.5 mm
- net VBUS: track 5.71 -> 8.31 mm
