File: X88H.kicad_pcb (KiCad board)
At the start: 2 copper layers, 344 x 124.1 mm, 251 parts, among them J1 SM04B-SRSS-TB, J2 TC2030_SWD, U1 XC6206P332MR, U2 STM32F072CBT6

Commit message: Rotate JST to face alphas
Parts:
- turned J1 to 90 degrees
Routing:
- net VBUS: track 40.2 -> 50.6 mm
- net D-: track 102.0 -> 109.3 mm
- net D+: track 101.7 -> 109.1 mm
- net GND: track 62.4 -> 56.9 mm, vias 150 -> 148
- net +5V: track 402.5 -> 403.0 mm
